File: main.sch (EAGLE design)
At the start: 11 parts, among them U1 XC7A35T-1FTG256C, U2 MT25QU128ABA1ESE

Commit message: Created new FPGA library
Parts:
- removed SJ3: (no value), jumper:SJ2W
- added JP1: (no value), jumper:JP1E
- added R6: (no value), rcl:R-EU_R0603
- U1: value XC7A35T-1FTG256C -> XC7A15T-1FTG256C; device XC7A35T-1FTG256C:XC7A35T-1FTG256C -> XC7A35T-1FTG256C:XC7A15T-1FTG256C
Connections:
- removed net N$3: U1.DONE_0
- net CCLK: now also U1G$2.CCLK_0; no longer U1.CCLK_0
- net CS: now also U1G$4.IO_L6P_T0_FCS_B_14; no longer U1.IO_L6P_T0_FCS_B_14
- net GND: now also R6.2, U1G$1.GND, U1G$1.VCCBATT_0, U1G$2.CFGBVS_0, U1G$2.DXN_0, U1G$2.DXP_0, U1G$4.IO_L3P_T0_DQS_PUDC_B_14; no longer SJ3.1, U1.CFGBVS_0, U1.DXN_0, U1.DXP_0, U1.GND, U1.GNDADC_0, U1.IO_L3P_T0_DQS_PUDC_B_14, U1.VCCBATT_0, U1.VN_0, U1.VP_0, U1.VREFN_0, U1.VREFP_0
- net HOLD: now also U1G$4.IO_L2N_T0_D03_14; no longer U1.IO_L2N_T0_D03_14
- net M0: now also U1G$2.M0_0; no longer U1.M0_0
- net M1: now also U1G$2.M1_0; no longer U1.M1_0
- net M2: now also JP1.2, R6.1, U1G$2.M2_0; no longer SJ3.2, U1.M2_0
- net MISO: now also U1G$4.IO_L1N_T0_D01_DIN_14; no longer U1.IO_L1N_T0_D01_DIN_14
- net MOSI: now also U1G$4.IO_L1P_T0_D00_MOSI_14; no longer U1.IO_L1P_T0_D00_MOSI_14
- net N$2: now also U1G$2.INIT_B_0; no longer U1.INIT_B_0
- net N$4: now also U1G$2.PROGRAM_B_0; no longer U1.PROGRAM_B_0
- net TCK: now also U1G$2.TCK_0; no longer U1.TCK_0
- net TDI: now also U1G$2.TDI_0; no longer U1.TDI_0
- net TDO: now also U1G$2.TDO_0; no longer U1.TDO_0
- net TMS: now also U1G$2.TMS_0; no longer U1.TMS_0
- net VCC: now also JP1.1, U1G$1.VCCAUX, U1G$1.VCCO_0, U1G$1.VCCO_14, U1G$1.VCCO_15, U1G$1.VCCO_34, U1G$1.VCCO_35; no longer SJ3.3, U1.VCCADC_0, U1.VCCAUX, U1.VCCO_0
- net VCCINT: now also U1G$1.VCCBRAM, U1G$1.VCCINT; no longer U1.VCCBRAM, U1.VCCINT
- net WP: now also U1G$4.IO_L2P_T0_D02_14; no longer U1.IO_L2P_T0_D02_14
Other:
- note added: "FPGA CONFIGURATION"
- note added: "MODE SELECTION"
- moved on the sheet: R1, R2, R3, R4, R5, S1, SJ1, SJ2, U2
