File: main.sch (EAGLE design)
At the start: 11 parts, among them U1 XC7A35T-1FTG256C, U2 MT25QU128ABA1ESE

Commit message: Added input protection
Parts:
- added C1: 0.22u, rcl:C-EUC0805
- added C2, C3: 10u, rcl:C-EUC0805
- added C4, C5: DNP, rcl:C-EUC0805
- added C6: 3.3n, rcl:C-EUC0805
- added J1: (no value), con-jack:DCJ0303
- added LED1: (no value), led:LEDCHIP-LED0805
- added R10: 137k, rcl:R-EU_R0805
- added R11: 22k, rcl:R-EU_R0805
- added R12: 1k, rcl:R-EU_R0805
- added R6: 453k, rcl:R-EU_R0805
- added R7: 1.37M, rcl:R-EU_R0805
- added R8: 162k, rcl:R-EU_R0805
- added R9: 33.2m, rcl:R-EU_R0805
- added TP1, TP2: TPB1,27, testpad:TPB1,27
- added U$1: LTC4368, LTC4368:LTC4368
- added U$2: FDS3992, FDS3992:FDS3992
- added U$3: MPZ2012S101AT000, MPZ2012S101AT000:MPZ2012S101AT000
Connections:
- new net +5V0_UNREG: C3.1, C4.1, C5.1, R12.2, TP2.TP, U$3.2
- new net N$1: U$2G$1.S, U$2G$2.S
- new net N$10: R10.1, R8.2, U$1.OV
- new net N$11: C1.1, U$1.RETRY
- new net N$12: R9.1, U$1.SENSE, U$2G$2.D
- new net N$13: LED1.A, R12.1
- new net N$14: TP1.TP, U$1.~FAULT
- new net N$15: C6.1, R11.2
- new net N$5: C2.1, R9.2, U$1.VOUT, U$3.1
- new net N$6: R11.1, U$1.GATE, U$2G$1.G, U$2G$2.G
- new net N$7: R10.2, R7.1, U$1.UV
- new net N$8: J1.1, R6.2, U$1.VIN, U$2G$1.D
- new net N$9: R6.1, R7.2, U$1.~SHDN
- net GND: now also C1.2, C2.2, C3.2, C4.2, C5.2, C6.2, J1.2, J1.3, LED1.C, R8.1, U$1.GND

Commit message: Changed to new fpga library
Parts:
- removed SJ3: (no value), jumper:SJ2W
- added C7: 100n, rcl:C-EUC0603
- added JP1: (no value), jumper:JP1E
- added R13: 1k, rcl:R-EU_R0603
- U1: value XC7A35T-1FTG256C -> XC7A15T-1FTG256C; device XC7A35T-1FTG256C:XC7A35T-1FTG256C -> XC7A35T-1FTG256C:XC7A15T-1FTG256C
Connections:
- removed net N$3: U1.DONE_0
- removed net VCCINT: U1.VCCBRAM, U1.VCCINT
- new net +1V0_FPGA: U1G$1.VCCBRAM, U1G$1.VCCINT
- new net +1V8: U1G$1.VCCAUX, U1G$1.VCCO_0, U1G$1.VCCO_14, U1G$1.VCCO_15, U1G$1.VCCO_34, U1G$1.VCCO_35
- net CCLK: now also U1G$2.CCLK_0; no longer U1.CCLK_0
- net CS: now also U1G$4.IO_L6P_T0_FCS_B_14; no longer U1.IO_L6P_T0_FCS_B_14
- net GND: now also C7.2, R13.1, U1G$1.GND, U1G$1.VCCBATT_0, U1G$2.CFGBVS_0, U1G$2.DXN_0, U1G$2.DXP_0, U1G$4.IO_L3P_T0_DQS_PUDC_B_14; no longer SJ3.1, U1.CFGBVS_0, U1.DXN_0, U1.DXP_0, U1.GND, U1.GNDADC_0, U1.IO_L3P_T0_DQS_PUDC_B_14, U1.VCCBATT_0, U1.VN_0, U1.VP_0, U1.VREFN_0, U1.VREFP_0
- net HOLD: now also U1G$4.IO_L2N_T0_D03_14; no longer U1.IO_L2N_T0_D03_14
- net M0: now also U1G$2.M0_0; no longer U1.M0_0
- net M1: now also U1G$2.M1_0; no longer U1.M1_0
- net M2: now also JP1.2, R13.2, U1G$2.M2_0; no longer SJ3.2, U1.M2_0
- net MISO: now also U1G$4.IO_L1N_T0_D01_DIN_14; no longer U1.IO_L1N_T0_D01_DIN_14
- net MOSI: now also U1G$4.IO_L1P_T0_D00_MOSI_14; no longer U1.IO_L1P_T0_D00_MOSI_14
- net N$2: now also U1G$2.INIT_B_0; no longer U1.INIT_B_0
- net N$4: now also U1G$2.PROGRAM_B_0; no longer U1.PROGRAM_B_0
- net TCK: now also U1G$2.TCK_0; no longer U1.TCK_0
- net TDI: now also U1G$2.TDI_0; no longer U1.TDI_0
- net TDO: now also U1G$2.TDO_0; no longer U1.TDO_0
- net TMS: now also U1G$2.TMS_0; no longer U1.TMS_0
- net VCC: now also C7.1, JP1.1; no longer SJ3.3, U1.VCCADC_0, U1.VCCAUX, U1.VCCO_0
- net WP: now also U1G$4.IO_L2P_T0_D02_14; no longer U1.IO_L2P_T0_D02_14
Other:
- note added: "FPGA CONFIGURATION"
- note added: "MODE SELECT"

Commit message: Added DDR3 memory
Parts:
- added C10, C8: 10n, rcl:C-EUC0603
- added C11, C9: 1u, rcl:C-EUC0603
- added C12, C13, C14, C15, C16, C17, C18, C19, C20, C21, C22, C23, C24, C25, C26, C27: 47n, rcl:C-EUC0603
- added R14, R15: 1k 1%, rcl:R-EU_R0603
- added R16: 240R 1%, rcl:R-EU_R0603
- added U3: MT41K128M16JT-125:K, MT41K128M16JT-125_K:MT41K128M16JT-125:K
Connections:
- removed net VCC: C7.1, JP1.1, R1.2, R2.2, R3.2, R4.2, R5.2, SJ1.3, SJ2.3, U2.VCC
- new net +1V5: C10.1, C11.1, C12.1, C13.1, C14.1, C15.1, C16.1, C17.1, C18.1, C19.1, C20.1, C21.1, C22.1, C23.1, C24.1, C25.1, C26.1, C27.1, R14.2, U3.VDD, U3.VDDQ
- new net N$16: R16.2, U3.ZQ
- new net N$3: C10.2, C11.2, C8.1, C9.1, R14.1, R15.2, U3.VREFCA, U3.VREFDQ
- new net U3_!CAS: U3.!CAS
- new net U3_!CS: U3.!CS
- new net U3_!RAS: U3.!RAS
- new net U3_!RESET: U3.!RESET
- new net U3_!WE: U3.!WE
- new net U3_A0: U3.A0
- new net U3_A1: U3.A1
- new net U3_A10/AP: U3.A10/AP
- new net U3_A11: U3.A11
- new net U3_A12/!BC: U3.A12/!BC
- new net U3_A13: U3.A13
- new net U3_A2: U3.A2
- new net U3_A3: U3.A3
- new net U3_A4: U3.A4
- new net U3_A5: U3.A5
- new net U3_A6: U3.A6
- new net U3_A7: U3.A7
- new net U3_A8: U3.A8
- new net U3_A9: U3.A9
- new net U3_BA0: U3.BA0
- new net U3_BA1: U3.BA1
- new net U3_BA2: U3.BA2
- new net U3_CKE: U3.CKE
- new net U3_CK_P: U3.CK
- new net U3_CP_N: U3.!CK
- new net U3_DQ0: U3.DQ0
- new net U3_DQ1: U3.DQ1
- new net U3_DQ10: U3.DQ10
- new net U3_DQ11: U3.DQ11
- new net U3_DQ12: U3.DQ12
- new net U3_DQ13: U3.DQ13
- new net U3_DQ14: U3.DQ14
- new net U3_DQ15: U3.DQ15
- new net U3_DQ2: U3.DQ2
- new net U3_DQ3: U3.DQ3
- new net U3_DQ4: U3.DQ4
- new net U3_DQ5: U3.DQ5
- new net U3_DQ6: U3.DQ6
- new net U3_DQ7: U3.DQ7
- new net U3_DQ8: U3.DQ8
- new net U3_DQ9: U3.DQ9
- new net U3_LDM: U3.LDM
- new net U3_LDQS_N: U3.!LDQS
- new net U3_LDQS_P: U3.LDQS
- new net U3_ODT: U3.ODT
- new net U3_UDM: U3.UDM
- new net U3_UDQS_N: U3.!UDQS
- new net U3_UDQS_P: U3.UDQS
- net +1V8: now also C7.1, JP1.1, R1.2, R2.2, R3.2, R4.2, R5.2, SJ1.3, SJ2.3, U2.VCC
- net GND: now also C12.2, C13.2, C14.2, C15.2, C16.2, C17.2, C18.2, C19.2, C20.2, C21.2, C22.2, C23.2, C24.2, C25.2, C26.2, C27.2, C8.2, C9.2, R15.1, R16.1, U3.VSS, U3.VSSQ
